Commit message: updated github user

File: aristo/aristo.urdf (robot description, URDF)
Before this commit: robot aristo-v1.0, 9 links, 8 joints
Links:
- link hand_base: geometry collision mesh filename=https://raw.githubusercontent.com/akim-jinsoo/robot-urdfs/r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; visual mesh filename=https://raw.githubusercontent.com/akim-jinsoo/robot-urdfs/r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
- link index_distal: geometry collision mesh filename=https://raw.githubusercontent.com/akim-jinsoo/robot-urdfs/r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; visual mesh filename=https://raw.githubusercontent.com/akim-jinsoo/robot-urdfs/r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
- link index_proximal: geometry collision mesh filename=https://raw.githubusercontent.com/akim-jinsoo/robot-urdfs/r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; visual mesh filename=https://raw.githubusercontent.com/akim-jinsoo/robot-urdfs/r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
- link middle_distal: geometry collision mesh filename=https://raw.githubusercontent.com/akim-jinsoo/robot-urdfs/r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; visual mesh filename=https://raw.githubusercontent.com/akim-jinsoo/robot-urdfs/r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
- link middle_proximal: geometry collision mesh filename=https://raw.githubusercontent.com/akim-jinsoo/robot-urdfs/r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; visual mesh filename=https://raw.githubusercontent.com/akim-jinsoo/robot-urdfs/r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
- link thumb_actuators: geometry collision mesh filename=https://raw.githubusercontent.com/akim-jinsoo/robot-urdfs/r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; visual mesh filename=https://raw.githubusercontent.com/akim-jinsoo/robot-urdfs/r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
- link thumb_distal: geometry collision mesh filename=https://raw.githubusercontent.com/akim-jinsoo/robot-urdfs/r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; visual mesh filename=https://raw.githubusercontent.com/akim-jinsoo/robot-urdfs/r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
- link thumb_metacarpal: geometry collision mesh filename=https://raw.githubusercontent.com/akim-jinsoo/robot-urdfs/r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; visual mesh filename=https://raw.githubusercontent.com/akim-jinsoo/robot-urdfs/r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
- link thumb_proximal: geometry collision mesh filename=https://raw.githubusercontent.com/akim-jinsoo/robot-urdfs/r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; visual mesh filename=https://raw.githubusercontent.com/akim-jinsoo/robot-urdfs/r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

File: plato/plato_v2.urdf (robot description, URDF)
Before this commit: robot plato2, 9 links, 8 joints
Links:
- link base_link: geometry collision mesh filename=https://raw.githubusercontent.com/akim-jinsoo/robot-urdfs/r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; visual mesh filename=https://raw.githubusercontent.com/akim-jinsoo/robot-urdfs/r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
- link index_distal: geometry collision mesh filename=https://raw.githubusercontent.com/akim-jinsoo/robot-urdfs/r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; visual mesh filename=https://raw.githubusercontent.com/akim-jinsoo/robot-urdfs/r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
- link index_proximal: geometry collision mesh filename=https://raw.githubusercontent.com/akim-jinsoo/robot-urdfs/r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; visual mesh filename=https://raw.githubusercontent.com/akim-jinsoo/robot-urdfs/r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
- link middle_distal: geometry collision mesh filename=https://raw.githubusercontent.com/akim-jinsoo/robot-urdfs/r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; visual mesh filename=https://raw.githubusercontent.com/akim-jinsoo/robot-urdfs/r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
- link middle_proximal: geometry collision mesh filename=https://raw.githubusercontent.com/akim-jinsoo/robot-urdfs/r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; visual mesh filename=https://raw.githubusercontent.com/akim-jinsoo/robot-urdfs/r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
- link thumb_actuators: geometry collision mesh filename=https://raw.githubusercontent.com/akim-jinsoo/robot-urdfs/r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; visual mesh filename=https://raw.githubusercontent.com/akim-jinsoo/robot-urdfs/r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
- link thumb_distal: geometry collision mesh filename=https://raw.githubusercontent.com/akim-jinsoo/robot-urdfs/r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; visual mesh filename=https://raw.githubusercontent.com/akim-jinsoo/robot-urdfs/r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
- link thumb_metacarpal: geometry collision mesh filename=https://raw.githubusercontent.com/akim-jinsoo/robot-urdfs/r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; visual mesh filename=https://raw.githubusercontent.com/akim-jinsoo/robot-urdfs/r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
- link thumb_proximal: geometry collision mesh filename=https://raw.githubusercontent.com/akim-jinsoo/robot-urdfs/r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; visual mesh filename=https://raw.githubusercontent.com/akim-jinsoo/robot-urdfs/r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
